File: CAD/100w BLDC MC PCB/100w BLDC Motor Controller Pathfinder/100w BLDC Motor Controller Pathfinder.kicad_sch (KiCad schematic)
At the start: 37 parts, among them J1 USB_C_Receptacle_USB2.0, SW1 PTS815 SJM 250 SMTR LFS, U1 RP2040, U2 W25Q128JVS, U3 USBLC6-2SC6, U4 LMR36506MSC3RPERQ1, Y1 ABLS-12.000MHZ-B4-T

Commit message: organización
Parts:
- removed C15, C18: 100n 50v, symbol Device:C
- removed C16: 2u2 50v, symbol Device:C
- removed C17: 1u 16v, symbol Device:C
- removed C19, C20: 22u, symbol Device:C
- removed D1, D2: DSS14UTR, DSS14UTR:SODFL3618X110N, symbol DSS14UTR:DSS14UTR
- removed J1: USB_C_Receptacle_USB2.0, symbol Connector:USB_C_Receptacle_USB2.0
- removed L1: 15L, symbol Device:L
- removed R6, R7: 1k5, symbol Device:R
- removed U3: USBLC6-2SC6, Package_TO_SOT_SMD:SOT-23-6, symbol Power_Protection:USBLC6-2SC6
- removed U4: LMR36506MSC3RPERQ1, RPE0009A, symbol 2024-01-23_05-03-01:LMR36506MSC3RPERQ1
Connections:
- no-connect marks 3 -> 0
Other:
- added sheet Communication Peripherals (CP.kicad_sch)
- added sheet Motor Driver & Encoder (MD.kicad_sch)
- added sheet Power (Power.kicad_sch)
- note removed: "Buck Switching Regulator"
- note removed: "USB"
- moved on the sheet: C12, C13, C14, R1, R2, R3, SW1, U2, Y1

Commit message: aun no
Connections:
- net Encoder_Z: now reaches U1.12 (GPIO9)
- net Encoder_MOSI: now reaches U1.2 (GPIO0)
- net Encoder_CS: now reaches U1.3 (GPIO1)
- net Encoder_SCLK: now reaches U1.4 (GPIO2)
- net Encoder_MISO: now reaches U1.5 (GPIO3)
- net Encoder_A: now reaches U1.7 (GPIO5)
- net Encoder_B: now reaches U1.9 (GPIO7)
Other:
- moved on the sheet: R4, R5
Changed lines of the file:
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@@
     (stroke (width 0) (type default))
   )
-  (wire (pts (xy 264.795 45.72) (xy 264.795 46.99))
+  (wire (pts (xy 264.16 45.72) (xy 264.16 46.99))
     (stroke (width 0) (type default))
   )
@@
     (stroke (width 0) (type dash_dot))
   )
-  (wire (pts (xy 264.795 46.99) (xy 257.81 46.99))
+  (wire (pts (xy 264.16 46.99) (xy 257.81 46.99))
     (stroke (width 0) (type default))
   )
@@
     (stroke (width 0) (type default))
   )
-  (wire (pts (xy 274.955 45.72) (xy 273.685 45.72))
+  (wire (pts (xy 274.32 45.72) (xy 273.05 45.72))
     (stroke (width 0) (type default))
   )
@@
     (stroke (width 0) (type default))
   )
+  (wire (pts (xy 179.07 24.13) (xy 179.07 18.415))
+    (stroke (width 0) (type default))
+  )
   (wire (pts (xy 38.1 99.06) (xy 55.245 99.06))
     (stroke (width 0) (type default))
@@
     (stroke (width 0) (type default))
   )
+  (wire (pts (xy 191.77 29.21) (xy 176.53 29.21))
+    (stroke (width 0) (type default))
+  )
   (wire (pts (xy 120.65 86.36) (xy 120.65 86.995))
     (stroke (width 0) (type default))
@@
     (stroke (width 0) (type default))
   )
-  (wire (pts (xy 264.795 49.53) (xy 257.81 49.53))
+  (wire (pts (xy 264.16 49.53) (xy 257.81 49.53))
     (stroke (width 0) (type default))
   )
@@
     (stroke (width 0) (type dash_dot))
   )
-  (wire (pts (xy 264.795 45.72) (xy 266.065 45.72))
+  (wire (pts (xy 264.16 45.72) (xy 265.43 45.72))
     (stroke (width 0) (type default))
   )
@@
     (stroke (width 0) (type default))
   )
+  (wire (pts (xy 180.34 15.24) (xy 167.64 15.24))
+    (stroke (width 0) (type default))
+  )
+  (wire (pts (xy 189.865 34.29) (xy 191.77 34.29))
+    (stroke (width 0) (type default))
+  )
   (wire (pts (xy 53.34 48.26) (xy 53.34 52.07))
     (stroke (width 0) (type default))
   )
+  (wire (pts (xy 191.77 21.59) (xy 180.34 21.59))
+    (stroke (width 0) (type default))
+  )
   (wire (pts (xy 259.08 39.37) (xy 257.81 39.37))
     (stroke (width 0) (type default))
   )
-  (wire (pts (xy 274.955 50.8) (xy 273.685 50.8))
+  (wire (pts (xy 274.32 50.8) (xy 273.05 50.8))
     (stroke (width 0) (type default))
   )
@@
     (stroke (width 0) (type dash_dot))
   )
-  (wire (pts (xy 266.065 50.8) (xy 264.795 50.8))
+  (wire (pts (xy 265.43 50.8) (xy 264.16 50.8))
     (stroke (width 0) (type default))
   )
@@
     (stroke (width 0) (type default))
   )
+  (wire (pts (xy 177.8 26.67) (xy 177.8 21.59))
+    (stroke (width 0) (type default))
+  )
   (wire (pts (xy 124.46 34.925) (xy 124.46 36.83))
     (stroke (width 0) (type default))
   )
+  (wire (pts (xy 180.34 21.59) (xy 180.34 15.24))
+    (stroke (width 0) (type default))
+  )
+  (wire (pts (xy 176.53 24.765) (xy 167.64 24.765))
+    (stroke (width 0) (type default))
+  )
   (wire (pts (xy 40.64 22.225) (xy 40.64 26.035))
     (stroke (width 0) (type default))
@@
     (stroke (width 0) (type default))
   )
+  (wire (pts (xy 191.77 24.13) (xy 179.07 24.13))
+    (stroke (width 0) (type default))
+  )
   (wire (pts (xy 60.96 48.26) (xy 63.5 48.26))
     (stroke (width 0) (type default))
   )
+  (wire (pts (xy 189.865 39.37) (xy 191.77 39.37))
+    (stroke (width 0) (type default))
+  )
   (polyline (pts (xy 66.04 134.62) (xy 65.405 134.62))
+    (stroke (width 0) (type default))
+  )
+  (wire (pts (xy 191.77 26.67) (xy 177.8 26.67))
     (stroke (width 0) (type default))
   )
@@
     (stroke (width 0) (type default))
   )
-  (wire (pts (xy 264.795 50.8) (xy 264.795 49.53))
+  (wire (pts (xy 264.16 50.8) (xy 264.16 49.53))
     (stroke (width 0) (type default))
   )
@@
     (stroke (width 0) (type default))
   )
+  (wire (pts (xy 177.8 21.59) (xy 167.64 21.59))
+    (stroke (width 0) (type default))
+  )
   (wire (pts (xy 40.64 48.26) (xy 40.64 52.07))
     (stroke (width 0) (type default))
   )
+  (wire (pts (xy 176.53 29.21) (xy 176.53 24.765))
+    (stroke (width 0) (type default))
+  )
   (wire (pts (xy 76.2 48.26) (xy 91.44 48.26))
     (stroke (width 0) (type default))
@@
   )
   (wire (pts (xy 78.74 99.06) (xy 78.74 104.14))
+    (stroke (width 0) (type default))
+  )
+  (wire (pts (xy 179.07 18.415) (xy 167.64 18.415))
     (stroke (width 0) (type default))
   )
@@
     (stroke (width 0) (type dash_dot))
   )
+  (wire (pts (xy 189.865 44.45) (xy 191.77 44.45))
+    (stroke (width 0) (type default))
+  )
   (wire (pts (xy 257.81 55.88) (xy 262.255 55.88))
     (stroke (width 0) (type default))
@@
     (effects (font (size 1.27 1.27)) (justify left bottom))
   )
-  (label "USB_D+" (at 274.955 50.8 0) (fields_autoplaced)
-    (effects (font (size 1.27 1.27)) (justify left bottom))
-  )
   (label "XOUT" (at 259.08 21.59 0) (fields_autoplaced)
     (effects (font (size 1.27 1.27)) (justify left bottom))
@@
     (effects (font (size 1.27 1.27)) (justify right bottom))
   )
-  (label "USB_D-" (at 274.955 45.72 0) (fields_autoplaced)
-    (effects (font (size 1.27 1.27)) (justify left bottom))
-  )
   (label "QSPI_SD0" (at 259.08 34.29 0) (fields_autoplaced)
     (effects (font (size 1.27 1.27)) (justify left bottom))
@@
   (label "QSPI_SD2" (at 106.68 111.76 180) (fields_autoplaced)
     (effects (font (size 1.27 1.27)) (justify right bottom))
+  )
+  (global_label "USB_D+" (shape input) (at 274.32 50.8 0) (fields_autoplaced)
+    (effects (font (size 1.27 1.27)) (justify left))
+    (property "Intersheetrefs" "${INTERSHEET_REFS}" (at 284.8458 50.8 0)
+      (effects (font (size 1.27 1.27)) (justify left) hide)
+    )
+  )
+  (global_label "Encoder_MOSI" (shape input) (at 167.64 15.24 180) (fields_autoplaced)
+    (effects (font (size 1.27 1.27)) (justify right))
+    (property "Intersheetrefs" "${INTERSHEET_REFS}" (at 151.611 15.24 0)
+      (effects (font (size 1.27 1.27)) (justify right) hide)
+    )
+  )
+  (global_label "Encoder_CS" (shape input) (at 167.64 18.415 180) (fields_autoplaced)
+    (effects (font (size 1.27 1.27)) (justify right))
+    (property "Intersheetrefs" "${INTERSHEET_REFS}" (at 153.7277 18.415 0)
+      (effects (font (size 1.27 1.27)) (justify right) hide)
+    )
+  )
+  (global_label "USB_D-" (shape input) (at 274.32 45.72 0) (fields_autoplaced)
+    (effects (font (size 1.27 1.27)) (justify left))
+    (property "Intersheetrefs" "${INTERSHEET_REFS}" (at 284.8458 45.72 0)
+      (effects (font (size 1.27 1.27)) (justify left) hide)
+    )
+  )
+  (global_label "Encoder_A" (shape input) (at 189.865 34.29 180) (fields_autoplaced)
+    (effects (font (size 1.27 1.27)) (justify right))
+    (property "Intersheetrefs" "${INTERSHEET_REFS}" (at 177.3436 34.29 0)
+      (effects (font (size 1.27 1.27)) (justify right) hide)
+    )
+  )
+  (global_label "Encoder_MISO" (shape input) (at 167.64 24.765 180) (fields_autoplaced)
+    (effects (font (size 1.27 1.27)) (justify right))
+    (property "Intersheetrefs" "${INTERSHEET_REFS}" (at 151.611 24.765 0)
+      (effects (font (size 1.27 1.27)) (justify right) hide)
+    )
+  )
+  (global_label "Encoder_B" (shape input) (at 189.865 39.37 180) (fields_autoplaced)
+    (effects (font (size 1.27 1.27)) (justify right))
+    (property "Intersheetrefs" "${INTERSHEET_REFS}" (at 177.1622 39.37 0)
+      (effects (font (size 1.27 1.27)) (justify right) hide)
+    )
+  )
+  (global_label "Encoder_Z" (shape input) (at 189.865 44.45 180) (fields_autoplaced)
+    (effects (font (size 1.27 1.27)) (justify right))
+    (property "Intersheetrefs" "${INTERSHEET_REFS}" (at 177.2227 44.45 0)
+      (effects (font (size 1.27 1.27)) (justify right) hide)
+    )
+  )
+  (global_label "Encoder_SCLK" (shape input) (at 167.64 21.59 180) (fields_autoplaced)
+    (effects (font (size 1.27 1.27)) (justify right))
+    (property "Intersheetrefs" "${INTERSHEET_REFS}" (at 151.4296 21.59 0)
+      (effects (font (size 1.27 1.27)) (justify right) hide)
+    )
   )
   (symbol (lib_id "2024-01-22_00-26-35:RP2040") (at 43.18 52.07 90) (mirror x) (unit 2)
@@
     )
   )
-  (symbol (lib_id "Device:R") (at 269.875 45.72 90) (unit 1)
+  (symbol (lib_id "Device:R") (at 269.24 45.72 90) (unit 1)
     (in_bom yes) (on_board yes) (dnp no)
-    (property "Reference" "R4" (at 266.065 44.45 90)
+    (property "Reference" "R4" (at 265.43 44.45 90)
       (effects (font (size 1.27 1.27)))
     )
-    (property "Value" "27Ω4" (at 269.875 43.18 90)
+    (property "Value" "27Ω4" (at 269.24 43.18 90)
       (effects (font (size 1.27 1.27)))
     )
-    (property "Footprint" "" (at 269.875 47.498 90)
-      (effects (font (size 1.27 1.27)) hide)
-    )
-    (property "Datasheet" "~" (at 269.875 45.72 0)
+    (property "Footprint" "" (at 269.24 47.498 90)
+      (effects (font (size 1.27 1.27)) hide)
+    )
+    (property "Datasheet" "~" (at 269.24 45.72 0)
       (effects (font (size 1.27 1.27)) hide)
     )
@@
     )
   )
-  (symbol (lib_id "Device:R") (at 269.875 50.8 90) (unit 1)
+  (symbol (lib_id "Device:R") (at 269.24 50.8 90) (unit 1)
     (in_bom yes) (on_board yes) (dnp no)
-    (property "Reference" "R5" (at 266.065 49.53 90)
+    (property "Reference" "R5" (at 265.43 49.53 90)
       (effects (font (size 1.27 1.27)))
     )
-    (property "Value" "27Ω4" (at 269.875 48.26 90)
+    (property "Value" "27Ω4" (at 269.24 48.26 90)
       (effects (font (size 1.27 1.27)))
     )
-    (property "Footprint" "" (at 269.875 52.578 90)
-      (effects (font (size 1.27 1.27)) hide)
-    )
-    (property "Datasheet" "~" (at 269.875 50.8 0)
-      (effects (font (size 1.27 1.27)) hide)
-    )
+    (property "Footprint" "" (at 269.24 52.578 90)
+      (effects (font (size 1.27 1.27)) hide)
+    )
+    (property "Datasheet" "~" (at 269.24 50.8 0)
+      (effects (font (size 1.27 1.27)) hide)
+    )

Commit message: Errores pero que probablemente no son errores
Parts:
- added C31, C32, C33: 100n, symbol Device:C
- added D3, D4, D5: WS2812B, LED_SMD:LED_WS2812B_PLCC4_5.0x5.0mm_P3.2mm, symbol LED:WS2812B
- added SW2: PTS815 SJM 250 SMTR LFS, SW4_PTS815 SJM 250 SMTR LFS_CNK, symbol 2024-01-22_02-04-17:PTS815_SJM_250_SMTR_LFS
Connections:
- net Encoder_MISO: now also U1.2 (GPIO0); no longer U1.5 (GPIO3)
- net Encoder_MOSI: now also U1.5 (GPIO3); no longer U1.2 (GPIO0)
- net GND: now also C31.2, C32.2, C33.2, D3.3 (VSS), D4.3 (VSS), D5.3 (VSS), SW2.1, SW2.2
- net GPIO8: now reaches U1.11 (GPIO8)
- net GPIO8: now also D3.4 (DIN)
- net GPIO10: now reaches U1.13 (GPIO10)
- net nFOULT: now reaches U1.14 (GPIO11)
- net DRV_SDO: now reaches U1.15 (GPIO12)
- net DRV_CS: now reaches U1.16 (GPIO13)
- net DRV_SCLK: now reaches U1.17 (GPIO14)
- net DRV_SDI: now reaches U1.18 (GPIO15)
- net SWCLK: now reaches U1.24 (SWCLK)
- net SWDIO: now reaches U1.25 (SWDIO)
- net at U1.26 (RUN): now also SW2.3, SW2.4
- net DRV_INLC: now reaches U1.27 (GPIO16)
- net DRV_INHC: now reaches U1.28 (GPIO17)
- net DRV_INLB: now reaches U1.29 (GPIO18)
- net DRV_INHB: now reaches U1.30 (GPIO19)
- net DRV_INLA: now reaches U1.31 (GPIO20)
- net DRV_INHA: now reaches U1.32 (GPIO21)
- net CAN_TX: now reaches U1.34 (GPIO22)
- net CAN_RX: now reaches U1.35 (GPIO23)
- net GPIO24: now reaches U1.36 (GPIO24)
- net GPIO25: now reaches U1.37 (GPIO25)
- net Batt_Voltage_Divider: now reaches U1.38 (GPIO26/ADC0)
- net DRV_SOA: now reaches U1.39 (GPIO27/ADC1)
- net DRV_SOB: now reaches U1.40 (GPIO28/ADC2)
- net DRV_SOC: now reaches U1.41 (GPIO29/ADC3)
- net DRVOFF: now reaches U1.6 (GPIO4)
- net VREF/ILIM: now reaches U1.8 (GPIO6)
- new net: D3.2 (DOUT), D4.4 (DIN)
- new net: D4.2 (DOUT), D5.4 (DIN)
- new net +5V: C31.1, C32.1, C33.1, D3.1 (VDD), D4.1 (VDD), D5.1 (VDD)
- no-connect marks 0 -> 1
Other:
- note added: "NeoPixels"

Commit message: ?
Changed lines of the file:
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@@
   (junction (at 124.46 25.4) (diameter 0) (color 0 0 0 0)
   )
-  (junction (at 88.265 48.26) (diameter 0) (color 0 0 0 0)
-  )
   (junction (at 17.78 36.83) (diameter 0) (color 0 0 0 0)
   )
@@
   )
   (junction (at 78.74 104.14) (diameter 0) (color 0 0 0 0)
+  )
+  (junction (at 24.13 149.86) (diameter 0) (color 0 0 0 0)
   )
   (junction (at 55.245 149.86) (diameter 0) (color 0 0 0 0)
@@
     (stroke (width 0) (type default))
   )
-  (wire (pts (xy 20.955 149.86) (xy 36.195 149.86))
+  (wire (pts (xy 20.955 149.86) (xy 24.13 149.86))
     (stroke (width 0) (type default))
   )
@@
     (stroke (width 0) (type default))
   )
-  (wire (pts (xy 88.265 47.625) (xy 88.265 48.26))
-    (stroke (width 0) (type default))
-  )
   (wire (pts (xy 78.74 25.4) (xy 90.17 25.4))
     (stroke (width 0) (type default))
@@
     (stroke (width 0) (type default))
   )
+  (wire (pts (xy 24.13 149.225) (xy 24.13 149.86))
+    (stroke (width 0) (type default))
+  )
   (wire (pts (xy 106.68 114.3) (xy 110.49 114.3))
     (stroke (width 0) (type default))
@@
     (stroke (width 0) (type default))
   )
-  (wire (pts (xy 88.265 48.26) (xy 91.44 48.26))
-    (stroke (width 0) (type default))
-  )
   (wire (pts (xy 259.08 39.37) (xy 257.81 39.37))
     (stroke (width 0) (type default))
@@
     (stroke (width 0) (type default))
   )
-  (wire (pts (xy 76.2 48.26) (xy 88.265 48.26))
+  (wire (pts (xy 76.2 48.26) (xy 91.44 48.26))
     (stroke (width 0) (type default))
   )
@@
   )
   (wire (pts (xy 189.865 59.69) (xy 191.77 59.69))
+    (stroke (width 0) (type default))
+  )
+  (wire (pts (xy 24.13 149.86) (xy 36.195 149.86))
     (stroke (width 0) (type default))
   )
@@
     )
   )
+  (symbol (lib_id "power:PWR_FLAG") (at 24.13 149.225 0) (unit 1)
+    (in_bom yes) (on_board yes) (dnp no) (fields_autoplaced)
+    (property "Reference" "#FLG02" (at 24.13 147.32 0)
+      (effects (font (size 1.27 1.27)) hide)
+    )
+    (property "Value" "PWR_FLAG" (at 24.13 144.78 0)
+      (effects (font (size 1.27 1.27)) hide)
+    )
+    (property "Footprint" "" (at 24.13 149.225 0)
+      (effects (font (size 1.27 1.27)) hide)
+    )
+    (property "Datasheet" "~" (at 24.13 149.225 0)
+      (effects (font (size 1.27 1.27)) hide)
+    )
+    (pin "1")
+    (instances
+      (project "100w BLDC Motor Controller Pathfinder"
+        (path "/bd5e620c-77b3-46f1-a718-89cd1182fd75"
+          (reference "#FLG02") (unit 1)
+        )
+      )
+    )
+  )
   (symbol (lib_id "2024-01-22_02-04-17:PTS815_SJM_250_SMTR_LFS") (at 73.66 97.79 0) (unit 1)
     (in_bom yes) (on_board yes) (dnp no)
@@
         )
       )
-    )
-  )
-  (symbol (lib_id "power:PWR_FLAG") (at 88.265 47.625 0) (unit 1)
-    (in_bom yes) (on_board yes) (dnp no) (fields_autoplaced)
-    (property "Reference" "#FLG02" (at 88.265 45.72 0)
-      (effects (font (size 1.27 1.27)) hide)
-    )
-    (property "Value" "PWR_FLAG" (at 88.265 43.18 0)
-      (effects (font (size 1.27 1.27)) hide)
-    )
-    (property "Footprint" "" (at 88.265 47.625 0)
-      (effects (font (size 1.27 1.27)) hide)
-    )
-    (property "Datasheet" "~" (at 88.265 47.625 0)
-      (effects (font (size 1.27 1.27)) hide)
-    )
-    (pin "1")
-    (instances
-      (project "100w BLDC Motor Controller Pathfinder"
-        (path "/bd5e620c-77b3-46f1-a718-89cd1182fd75/86cdd35b-a858-4f37-a673-ec7a499e55c2"
-          (reference "#FLG02") (unit 1)
-        )
-        (path "/bd5e620c-77b3-46f1-a718-89cd1182fd75"
-          (reference "#FLG05") (unit 1)
-        )
-      )

Commit message: Rev: 0.1
Parts:
- added C43: 100n, symbol Device:C
- added R13: 1k, symbol Device:R
- added R8: 10k, symbol Device:R
- added SW3: PTS815 SJM 250 SMTR LFS, SW4_PTS815 SJM 250 SMTR LFS_CNK, symbol 2024-01-22_02-04-17:PTS815_SJM_250_SMTR_LFS
Connections:
- net Encoder_A is gone; now on net CAN_RX: U1.7 (GPIO5)
- net +3V3: now also SW3.1, SW3.2
- net CAN_RX: no longer U1.35 (GPIO23)
- net CAN_TX: now also U1.6 (GPIO4); no longer U1.34 (GPIO22)
- net DRVOFF: now also U1.34 (GPIO22); no longer U1.6 (GPIO4)
- net GND: now also C43.2, R8.2
- net GPIO10: now also D3.4 (DIN)
- net RUN: now reaches SW2.3, SW2.4, U1.26 (RUN)
- net Encoder_B renamed GPIO7
- net GPIO7: now also C43.1, R13.2, R8.1
- net Encoder_Z renamed UART_RX
- net GPIO8 renamed UART_TX
- net UART_TX: no longer D3.4 (DIN)
- new net: R13.1, SW3.3, SW3.4
- new net GPIO23: U1.35 (GPIO23)
Other:
- note added: "RUN button"
- note added: "User button"
- company: (none) -> SCS
- title: (none) -> 100w BLDC Motor Controller Pathfinder
- moved on the sheet: SW2
