File: CAD/100w BLDC MC PCB/100w BLDC Motor Controller Pathfinder/MD.kicad_sch (KiCad schematic)
At the start: 0 parts

Commit message: poquito a poquito
Parts:
- added U5: MA704GQ-P, QFN-3x3_MA704_MNP, symbol 2024-02-01_06-45-48:MA704GQ-P
- added U6: DRV8316CRRGFR, VQFN40_RGF_TEX, symbol 2024-02-01_06-48-08:DRV8316CRRGFR
Changed lines of the file:
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@@
 (kicad_sch (version 20230121) (generator eeschema)
   (paper "A4")
+  (symbol (lib_id "2024-02-01_06-48-08:DRV8316CRRGFR") (at 64.135 58.42 0) (unit 1)
+    (in_bom yes) (on_board yes) (dnp no)
+    (property "Reference" "U6" (at 109.855 52.07 0)
+      (effects (font (size 1.524 1.524)))
+    )
+    (property "Value" "DRV8316CRRGFR" (at 102.235 113.03 0)
+      (effects (font (size 1.524 1.524)))
+    )
+    (property "Footprint" "VQFN40_RGF_TEX" (at 64.135 58.42 0)
+      (effects (font (size 1.27 1.27) italic) hide)
+    )
+    (property "Datasheet" "DRV8316CRRGFR" (at 62.865 54.61 0)
+      (effects (font (size 1.27 1.27) italic) hide)
+    )
+    (pin "1")
+    (pin "10")
+    (pin "11")
+    (pin "12")
+    (pin "13")
+    (pin "14")
+    (pin "15")
+    (pin "16")
+    (pin "17")
+    (pin "18")
+    (pin "19")
+    (pin "2")
+    (pin "20")
+    (pin "21")
+    (pin "22")
+    (pin "23")
+    (pin "24")
+    (pin "25")
+    (pin "26")
+    (pin "27")
+    (pin "28")
+    (pin "29")
+    (pin "3")
+    (pin "30")
+    (pin "31")
+    (pin "32")
+    (pin "33")
+    (pin "34")
+    (pin "35")
+    (pin "36")
+    (pin "37")
+    (pin "38")
+    (pin "39")
+    (pin "4")
+    (pin "40")
+    (pin "41")
+    (pin "5")
+    (pin "6")
+    (pin "7")
+    (pin "8")
+    (pin "9")
+    (instances
+      (project "100w BLDC Motor Controller Pathfinder"
+        (path "/bd5e620c-77b3-46f1-a718-89cd1182fd75/c4ad5e8b-cc6a-4605-ae3c-e9a1e8ea3baf"
+          (reference "U6") (unit 1)
+        )
+      )
+    )
+  )
+  (symbol (lib_id "2024-02-01_06-45-48:MA704GQ-P") (at 209.55 75.565 0) (unit 1)
+    (in_bom yes) (on_board yes) (dnp no)
+    (property "Reference" "U5" (at 240.665 69.215 0)
+      (effects (font (size 1.524 1.524)))
+    )
+    (property "Value" "MA704GQ-P" (at 234.95 109.22 0)
+      (effects (font (size 1.524 1.524)))
+    )
+    (property "Footprint" "QFN-3x3_MA704_MNP" (at 205.74 71.755 0)
+      (effects (font (size 1.27 1.27) italic) hide)
+    )
+    (property "Datasheet" "MA704GQ-P" (at 223.52 69.215 0)
+      (effects (font (size 1.27 1.27) italic) hide)
+    )
+    (pin "1")
+    (pin "10")
+    (pin "11")
+    (pin "12")
+    (pin "13")
+    (pin "14")
+    (pin "15")
+    (pin "16")
+    (pin "17")
+    (pin "2")
+    (pin "3")
+    (pin "4")
+    (pin "5")
+    (pin "6")
+    (pin "7")
+    (pin "8")
+    (pin "9")
+    (instances
+      (project "100w BLDC Motor Controller Pathfinder"
+        (path "/bd5e620c-77b3-46f1-a718-89cd1182fd75/c4ad5e8b-cc6a-4605-ae3c-e9a1e8ea3baf"
+          (reference "U5") (unit 1)
+        )
+      )
+    )
+  )
 )

Commit message: aun no
Parts:
- added C21: 1u, symbol Device:C
- added C22, C28: 1u 16v, symbol Device:C
- added C23: 10u 63v, symbol Device:C
- added C24: 2u2 63v, symbol Device:C
- added C25: 47n 63v, symbol Device:C
- added C26: 22u 10v, symbol Device:C
- added C27: 100n 63v, symbol Device:C
- added R8: 22, symbol Device:R
- added R9: 5k1, symbol Device:R
Connections:
- net +BATT: now reaches U6.10 (VM)
- net +BATT: now also U6.11 (VM), U6.9 (VM), C22.1, C23.1, C24.1
- net GND: now reaches U6.12 (PGND)
- net GND: now also U5.10 (TEST), U5.17 (PAD), U5.8 (GND), U6.15 (PGND), U6.18 (PGND), U6.2 (AGND), U6.26 (AGND), U6.4 (GND_BK), U6.41 (EPAD), C21.2, C23.2, C24.2, C26.2, C27.2, C28.2
- net Motor_A: now reaches U6.13 (OUTA)
- net Motor_A: now also U6.14 (OUTA)
- net Motor_B: now reaches U6.16 (OUTB)
- net Motor_B: now also U6.17 (OUTB)
- net Motor_C: now reaches U6.19 (OUTC)
- net Motor_C: now also U6.20 (OUTC)
- net DRVOFF: now reaches U6.21 (DRVOFF)
- net nFOULT: now reaches U6.22 (NFAULT)
- net nFOULT: now also R9.2
- net +3.3V: now reaches U6.23 (NSLEEP)
- net +3.3V: now also R9.1
- net +3.3VADC: now reaches U6.25 (AVDD)
- net +3.3VADC: now also C28.1
- net DRV_INHA: now reaches U6.27 (INHA)
- net DRV_INLA: now reaches U6.28 (INLA)
- net DRV_INHB: now reaches U6.29 (INHB)
- net +5V: now reaches U6.3 (FB_BK)
- net +5V: now also C26.1, R8.1
- net DRV_INLB: now reaches U6.30 (INLB)
- net DRV_INHC: now reaches U6.31 (INHC)
- net DRV_INLC: now reaches U6.32 (INLC)
- net DRV_SDO: now reaches U6.33 (SDO)
- net DRV_SDI: now reaches U6.34 (SDI)
- net DRV_SCLK: now reaches U6.35 (SCLK)
- net DRV_CS: now reaches U6.36 (NSCS)
- net VREF/ILIM: now reaches U6.37 (VREF/ILIM)
- net VREF/ILIM: now also C27.1
- net DRV_SOC: now reaches U6.38 (SOC)
- net DRV_SOB: now reaches U6.39 (SOB)
- net DRV_SOA: now reaches U6.40 (SOA)
- net at U6.5 (SW_BK): now also R8.2
- net at U6.6 (CPL): now also C25.2
- net at U6.7 (CPH): now also C25.1
- net at U6.8 (CP): now also C22.2
- net Encoder_SCLK: now reaches U5.12 (SCLK)
- net +3V3: now reaches U5.13 (VDD)
- net +3V3: now also C21.1
- net Encoder_A: now reaches U5.2 (A)
- net Encoder_Z: now reaches U5.3 (Z)
- net Encoder_MOSI: now reaches U5.4 (MOSI)
- net Encoder_CS: now reaches U5.5 (CS)
- net Encoder_B: now reaches U5.6 (B)
- net Encoder_MISO: now reaches U5.7 (MISO)
- no-connect marks 0 -> 5
Other:
- note added: "Mag Encoder"
- note added: "Motor Driver"
- moved on the sheet: U5, U6

Commit message: Errores pero que probablemente no son errores
Parts:
- removed R8: 22, symbol Device:R
- added H1, H2, H3: MountingHole_Pad, MountingHole:MountingHole_3mm_Pad_TopBottom, symbol Mechanical:MountingHole_Pad
- added L2: 47uH, symbol Device:L
Connections:
- net +5V: now also L2.1
- net Motor_A: now also H1.1
- net Motor_B: now also H3.1
- net Motor_C: now also H2.1
- net at U6.5 (SW_BK): now also L2.2

Commit message: ?
Other:
- moved on the sheet: C22
Changed lines of the file:
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@@
   (junction (at 73.66 58.42) (diameter 0) (color 0 0 0 0)
   )
-  (junction (at 50.8 46.355) (diameter 0) (color 0 0 0 0)
-  )
   (junction (at 209.55 99.695) (diameter 0) (color 0 0 0 0)
   )
@@
   )
   (junction (at 49.53 104.775) (diameter 0) (color 0 0 0 0)
-  )
-  (junction (at 21.59 84.455) (diameter 0) (color 0 0 0 0)
   )
   (junction (at 76.2 58.42) (diameter 0) (color 0 0 0 0)
@@
     (stroke (width 0) (type default))
   )
-  (wire (pts (xy 50.8 46.355) (xy 52.705 46.355))
+  (wire (pts (xy 81.28 55.88) (xy 81.28 60.325))
+    (stroke (width 0) (type default))
+  )
+  (wire (pts (xy 48.895 46.355) (xy 52.705 46.355))
     (stroke (width 0) (type default))
   )
@@
     (stroke (width 0) (type default))
   )
-  (wire (pts (xy 21.59 84.455) (xy 24.765 84.455))
-    (stroke (width 0) (type default))
-  )
-  (wire (pts (xy 21.59 83.185) (xy 21.59 84.455))
+  (wire (pts (xy 18.415 84.455) (xy 24.765 84.455))
     (stroke (width 0) (type default))
   )
@@
     (stroke (width 0) (type default))
   )
-  (wire (pts (xy 81.28 46.355) (xy 81.28 47.625))
+  (wire (pts (xy 81.28 46.355) (xy 81.28 48.26))
     (stroke (width 0) (type default))
   )
@@
     (stroke (width 0) (type default))
   )
-  (wire (pts (xy 48.895 46.355) (xy 50.8 46.355))
-    (stroke (width 0) (type default))
-  )
   (wire (pts (xy 153.035 105.41) (xy 153.035 106.68))
     (stroke (width 0) (type default))
@@
     (stroke (width 0) (type default))
   )
-  (wire (pts (xy 50.8 45.72) (xy 50.8 46.355))
-    (stroke (width 0) (type default))
-  )
   (wire (pts (xy 110.49 81.915) (xy 111.76 81.915))
     (stroke (width 0) (type default))
@@
   )
   (wire (pts (xy 52.705 57.15) (xy 52.705 55.245))
-    (stroke (width 0) (type default))
-  )
-  (wire (pts (xy 18.415 84.455) (xy 21.59 84.455))
-    (stroke (width 0) (type default))
-  )
-  (wire (pts (xy 81.28 55.245) (xy 81.28 60.325))
     (stroke (width 0) (type default))
   )
@@
     )
   )
-  (symbol (lib_id "power:PWR_FLAG") (at 21.59 83.185 0) (unit 1)
-    (in_bom yes) (on_board yes) (dnp no) (fields_autoplaced)
-    (property "Reference" "#FLG02" (at 21.59 81.28 0)
-      (effects (font (size 1.27 1.27)) hide)
-    )
-    (property "Value" "PWR_FLAG" (at 21.59 78.74 0)
-      (effects (font (size 1.27 1.27)) hide)
-    )
-    (property "Footprint" "" (at 21.59 83.185 0)
-      (effects (font (size 1.27 1.27)) hide)
-    )
-    (property "Datasheet" "~" (at 21.59 83.185 0)
-      (effects (font (size 1.27 1.27)) hide)
-    )
-    (pin "1")
-    (instances
-      (project "100w BLDC Motor Controller Pathfinder"
-        (path "/bd5e620c-77b3-46f1-a718-89cd1182fd75/86cdd35b-a858-4f37-a673-ec7a499e55c2"
-          (reference "#FLG02") (unit 1)
-        )
-        (path "/bd5e620c-77b3-46f1-a718-89cd1182fd75/c4ad5e8b-cc6a-4605-ae3c-e9a1e8ea3baf"
-          (reference "#FLG04") (unit 1)
-        )
-      )
-    )
-  )
   (symbol (lib_id "Device:C") (at 203.2 90.805 0) (unit 1)
     (in_bom yes) (on_board yes) (dnp no) (fields_autoplaced)
@@
     )
   )
-  (symbol (lib_id "Device:C") (at 81.28 51.435 0) (unit 1)
-    (in_bom yes) (on_board yes) (dnp no)
-    (property "Reference" "C22" (at 81.915 49.53 0)
-      (effects (font (size 1.27 1.27)) (justify left))
-    )
-    (property "Value" "1u 16v" (at 81.28 53.34 0)
-      (effects (font (size 1.27 1.27)) (justify left))
-    )
-    (property "Footprint" "" (at 82.2452 55.245 0)
-      (effects (font (size 1.27 1.27)) hide)
-    )
-    (property "Datasheet" "~" (at 81.28 51.435 0)
+  (symbol (lib_id "Device:C") (at 81.28 52.07 0) (unit 1)
+    (in_bom yes) (on_board yes) (dnp no)
+    (property "Reference" "C22" (at 81.915 50.165 0)
+      (effects (font (size 1.27 1.27)) (justify left))
+    )
+    (property "Value" "1u 16v" (at 81.28 53.975 0)
+      (effects (font (size 1.27 1.27)) (justify left))
+    )
+    (property "Footprint" "" (at 82.2452 55.88 0)
+      (effects (font (size 1.27 1.27)) hide)
+    )
+    (property "Datasheet" "~" (at 81.28 52.07 0)
       (effects (font (size 1.27 1.27)) hide)
     )
@@
     )
   )
-  (symbol (lib_id "power:PWR_FLAG") (at 50.8 45.72 0) (unit 1)
-    (in_bom yes) (on_board yes) (dnp no) (fields_autoplaced)
-    (property "Reference" "#FLG02" (at 50.8 43.815 0)
-      (effects (font (size 1.27 1.27)) hide)
-    )
-    (property "Value" "PWR_FLAG" (at 50.8 41.275 0)
-      (effects (font (size 1.27 1.27)) hide)
-    )
-    (property "Footprint" "" (at 50.8 45.72 0)
-      (effects (font (size 1.27 1.27)) hide)
-    )
-    (property "Datasheet" "~" (at 50.8 45.72 0)
-      (effects (font (size 1.27 1.27)) hide)
-    )
-    (pin "1")
-    (instances
-      (project "100w BLDC Motor Controller Pathfinder"
-        (path "/bd5e620c-77b3-46f1-a718-89cd1182fd75/86cdd35b-a858-4f37-a673-ec7a499e55c2"
-          (reference "#FLG02") (unit 1)
-        )
-        (path "/bd5e620c-77b3-46f1-a718-89cd1182fd75/c4ad5e8b-cc6a-4605-ae3c-e9a1e8ea3baf"
-          (reference "#FLG06") (unit 1)
-        )
-      )
-    )
-  )
   (symbol (lib_id "2024-02-01_06-48-08:DRV8316CRRGFR") (at 54.61 73.025 0) (unit 1)
     (in_bom yes) (on_board yes) (dnp no)
@@
       (effects (font (size 1.524 1.524)))
     )
-    (property "Footprint" "VQFN40_RGF_TEX" (at 54.61 74.295 0)
+    (property "Footprint" "VQFN40_RGF_TEX" (at 53.34 69.215 0)
       (effects (font (size 1.27 1.27) italic) hide)
     )
@@
     (pin "10")
     (pin "11")
+    (pin "21")
+    (pin "22")
+    (pin "23")
+    (pin "24")
+    (pin "27")
+    (pin "28")
+    (pin "29")
+    (pin "30")
+    (pin "31")
+    (pin "32")
+    (pin "33")
+    (pin "34")
+    (pin "35")
+    (pin "36")
+    (pin "38")
+    (pin "39")
+    (pin "40")
+    (pin "8")
+    (pin "9")
     (pin "12")
     (pin "13")
@@
     (pin "2")
     (pin "20")
-    (pin "21")
-    (pin "22")
-    (pin "23")
-    (pin "24")
     (pin "25")
     (pin "26")
-    (pin "27")
-    (pin "28")
-    (pin "29")
     (pin "3")
-    (pin "30")
-    (pin "31")
-    (pin "32")
-    (pin "33")
-    (pin "34")
-    (pin "35")
-    (pin "36")
     (pin "37")
-    (pin "38")
-    (pin "39")
     (pin "4")
-    (pin "40")
     (pin "41")
     (pin "5")
-    (pin "8")
-    (pin "9")
     (pin "6")
     (pin "7")
@@
     )
     (pin "1")
-    (pin "10")
     (pin "11")
     (pin "12")
@@
     (pin "8")
     (pin "9")
-    (instances
-      (project "100w BLDC Motor Controller Pathfinder"
+    (pin "10")
+    (instances
+      (project "100w BLDC Motor Controller Pathfinder"

Commit message: Rev: 0.1
Parts:
- removed C24: 2u2 63v, symbol Device:C
- added C16: 100n 63v, symbol Device:C
Connections:
- net +BATT: now also C16.1
- net GND: now also C16.2
- net Encoder_A: no longer names the net of U5.2 (A)
- net Encoder_B: no longer names the net of U5.6 (B)
- net Encoder_Z: no longer names the net of U5.3 (Z)
- no-connect marks 5 -> 8
Other:
- note added: "Motor Terminals"
- company: (none) -> SCS
- title: (none) -> 100w BLDC Motor Controller Pathfinder
- moved on the sheet: C21, C22, C23, C25, C26, C27, C28, H1, H2, H3, L2, R9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
