File: CAD/100w BLDC MC PCB/100w BLDC Motor Controller Pathfinder/Power.kicad_sch (KiCad schematic)
At the start: 10 parts, among them U4 LMR36506MSC3RPERQ1

Commit message: aun no
Parts:
- C15: value 2u2 50v -> 2u2 63v
- C16, C18: value 100n 50v -> 100n 63v
Changed lines of the file:
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@@
       (effects (font (size 1.27 1.27)) (justify left))
     )
-    (property "Value" "2u2 50v" (at 36.83 99.06 0)
+    (property "Value" "2u2 63v" (at 36.83 99.06 0)
       (effects (font (size 1.27 1.27)) (justify left))
     )
@@
       (effects (font (size 1.27 1.27)))
     )
-    (property "Value" "100n 50v" (at 101.6 86.36 90)
+    (property "Value" "100n 63v" (at 101.6 86.36 90)
       (effects (font (size 1.27 1.27)))
     )
@@
       (effects (font (size 1.27 1.27)) (justify left))
     )
-    (property "Value" "100n 50v" (at 47.625 99.06 0)
-      (effects (font (size 1.27 1.27)) (justify left))
-    )
+    (property "Value" "100n 63v" (at 47.625 99.06 0)
+      (effects (font (size 1.27 1.27)) (justify left))
+    )

Commit message: Errores pero que probablemente no son errores
Parts:
- added C23 (x9): 10u 63v, symbol Device:C
- added J8: Conn_01x02, Connector_AMASS:AMASS_XT30U-F_1x02_P5.0mm_Vertical, symbol Connector_Generic:Conn_01x02
- added R10: 110k, symbol Device:R
- added R11: 10k, symbol Device:R
- C19, C20: value 22u -> 22u 10v
- L1: value 15L -> 15uH
Connections:
- net +BATT: now also C23.1, C23.1, C23.1, C23.1, C23.1, C23.1, C23.1, C23.1, C23.1, J8.2 (Pin_2), R10.1
- net GND: now also C23.2, C23.2, C23.2, C23.2, C23.2, C23.2, C23.2, C23.2, C23.2, J8.1 (Pin_1), R11.1
- new net Batt_Voltage_Divider: R10.2, R11.2
Other:
- note added: "40v = 3.33v"
- note added: "Vmax = 32v (8s lipo)"
- note added: "Voltage Dicider"

Commit message: ?
Changed lines of the file:
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@@
   (junction (at 35.56 90.805) (diameter 0) (color 0 0 0 0)
   )
+  (junction (at 52.705 90.805) (diameter 0) (color 0 0 0 0)
+  )
   (junction (at 120.65 40.005) (diameter 0) (color 0 0 0 0)
   )
-  (junction (at 85.725 43.815) (diameter 0) (color 0 0 0 0)
-  )
   (junction (at 139.7 40.005) (diameter 0) (color 0 0 0 0)
   )
@@
   (junction (at 121.92 95.885) (diameter 0) (color 0 0 0 0)
   )
-  (junction (at 85.725 46.355) (diameter 0) (color 0 0 0 0)
+  (junction (at 86.36 43.815) (diameter 0) (color 0 0 0 0)
   )
   (junction (at 35.56 106.045) (diameter 0) (color 0 0 0 0)
@@
     (stroke (width 0) (type default))
   )
-  (wire (pts (xy 85.725 46.355) (xy 89.535 46.355))
-    (stroke (width 0) (type default))
-  )
   (wire (pts (xy 139.7 40.005) (xy 139.7 41.275))
     (stroke (width 0) (type default))
@@
     (stroke (width 0) (type default))
   )
+  (wire (pts (xy 52.705 90.805) (xy 58.42 90.805))
+    (stroke (width 0) (type default))
+  )
   (wire (pts (xy 92.71 40.005) (xy 102.235 40.005))
     (stroke (width 0) (type default))
@@
     (stroke (width 0) (type default))
   )
+  (wire (pts (xy 52.705 89.535) (xy 52.705 90.805))
+    (stroke (width 0) (type default))
+  )
   (wire (pts (xy 158.115 40.005) (xy 167.64 40.005))
     (stroke (width 0) (type default))
@@
     (stroke (width 0) (type default))
   )
+  (wire (pts (xy 86.36 43.815) (xy 89.535 43.815))
+    (stroke (width 0) (type default))
+  )
   (wire (pts (xy 130.175 40.005) (xy 139.7 40.005))
     (stroke (width 0) (type default))
@@
     (stroke (width 0) (type default))
   )
-  (wire (pts (xy 83.185 46.355) (xy 85.725 46.355))
+  (wire (pts (xy 83.185 46.355) (xy 89.535 46.355))
     (stroke (width 0) (type default))
   )
@@
     (stroke (width 0) (type default))
   )
+  (wire (pts (xy 80.01 125.73) (xy 80.01 124.46))
+    (stroke (width 0) (type default))
+  )
   (wire (pts (xy 111.76 40.005) (xy 120.65 40.005))
     (stroke (width 0) (type default))
@@
     (stroke (width 0) (type default))
   )
-  (wire (pts (xy 85.725 42.545) (xy 85.725 43.815))
-    (stroke (width 0) (type default))
-  )
   (wire (pts (xy 46.355 100.33) (xy 46.355 102.235))
     (stroke (width 0) (type default))
@@
     (stroke (width 0) (type default))
   )
+  (wire (pts (xy 86.36 42.545) (xy 86.36 43.815))
+    (stroke (width 0) (type default))
+  )
   (wire (pts (xy 120.015 116.205) (xy 120.015 124.46))
     (stroke (width 0) (type default))
@@
     (stroke (width 0) (type default))
   )
-  (wire (pts (xy 85.725 46.355) (xy 85.725 47.625))
-    (stroke (width 0) (type default))
-  )
   (wire (pts (xy 120.65 41.275) (xy 120.65 40.005))
     (stroke (width 0) (type default))
@@
     (stroke (width 0) (type default))
   )
-  (wire (pts (xy 83.185 43.815) (xy 85.725 43.815))
-    (stroke (width 0) (type default))
-  )
   (wire (pts (xy 120.65 48.895) (xy 120.65 50.8))
     (stroke (width 0) (type default))
@@
     (stroke (width 0) (type default))
   )
-  (wire (pts (xy 85.725 43.815) (xy 89.535 43.815))
+  (wire (pts (xy 83.185 43.815) (xy 86.36 43.815))
     (stroke (width 0) (type default))
   )
@@
     (stroke (width 0) (type default))
   )
-  (wire (pts (xy 46.355 90.805) (xy 58.42 90.805))
+  (wire (pts (xy 46.355 90.805) (xy 52.705 90.805))
     (stroke (width 0) (type default))
   )
@@
         (path "/bd5e620c-77b3-46f1-a718-89cd1182fd75/86cdd35b-a858-4f37-a673-ec7a499e55c2"
           (reference "L1") (unit 1)
-        )
-      )
-    )
-  )
-  (symbol (lib_id "power:GNDPWR") (at 85.725 47.625 0) (unit 1)
-    (in_bom yes) (on_board yes) (dnp no) (fields_autoplaced)
-    (property "Reference" "#PWR046" (at 85.725 52.705 0)
-      (effects (font (size 1.27 1.27)) hide)
-    )
-    (property "Value" "GNDPWR" (at 85.598 51.435 0)
-      (effects (font (size 1.27 1.27)) hide)
-    )
-    (property "Footprint" "" (at 85.725 48.895 0)
-      (effects (font (size 1.27 1.27)) hide)
-    )
-    (property "Datasheet" "" (at 85.725 48.895 0)
-      (effects (font (size 1.27 1.27)) hide)
-    )
-    (pin "1")
-    (instances
-      (project "100w BLDC Motor Controller Pathfinder"
-        (path "/bd5e620c-77b3-46f1-a718-89cd1182fd75/86cdd35b-a858-4f37-a673-ec7a499e55c2"
-          (reference "#PWR046") (unit 1)
         )
       )
@@
     )
   )
-  (symbol (lib_id "power:GND") (at 80.01 124.46 0) (unit 1)
-    (in_bom yes) (on_board yes) (dnp no) (fields_autoplaced)
-    (property "Reference" "#PWR020" (at 80.01 130.81 0)
-      (effects (font (size 1.27 1.27)) hide)
-    )
-    (property "Value" "GND" (at 80.01 128.905 0)
-      (effects (font (size 1.27 1.27)) hide)
-    )
-    (property "Footprint" "" (at 80.01 124.46 0)
-      (effects (font (size 1.27 1.27)) hide)
-    )
-    (property "Datasheet" "" (at 80.01 124.46 0)
+  (symbol (lib_id "power:GND") (at 80.01 125.73 0) (unit 1)
+    (in_bom yes) (on_board yes) (dnp no) (fields_autoplaced)
+    (property "Reference" "#PWR020" (at 80.01 132.08 0)
+      (effects (font (size 1.27 1.27)) hide)
+    )
+    (property "Value" "GND" (at 80.01 130.175 0)
+      (effects (font (size 1.27 1.27)) hide)
+    )
+    (property "Footprint" "" (at 80.01 125.73 0)
+      (effects (font (size 1.27 1.27)) hide)
+    )
+    (property "Datasheet" "" (at 80.01 125.73 0)
       (effects (font (size 1.27 1.27)) hide)
     )
@@
     )
   )
-  (symbol (lib_id "power:PWR_FLAG") (at 85.725 42.545 0) (unit 1)
-    (in_bom yes) (on_board yes) (dnp no) (fields_autoplaced)
-    (property "Reference" "#FLG02" (at 85.725 40.64 0)
-      (effects (font (size 1.27 1.27)) hide)
-    )
-    (property "Value" "PWR_FLAG" (at 85.725 38.1 0)
-      (effects (font (size 1.27 1.27)) hide)
-    )
-    (property "Footprint" "" (at 85.725 42.545 0)
-      (effects (font (size 1.27 1.27)) hide)
-    )
-    (property "Datasheet" "~" (at 85.725 42.545 0)
-      (effects (font (size 1.27 1.27)) hide)
-    )
-    (pin "1")
-    (instances
-      (project "100w BLDC Motor Controller Pathfinder"
-        (path "/bd5e620c-77b3-46f1-a718-89cd1182fd75/86cdd35b-a858-4f37-a673-ec7a499e55c2"
+  (symbol (lib_id "power:PWR_FLAG") (at 52.705 89.535 0) (unit 1)
+    (in_bom yes) (on_board yes) (dnp no) (fields_autoplaced)
+    (property "Reference" "#FLG02" (at 52.705 87.63 0)
+      (effects (font (size 1.27 1.27)) hide)
+    )
+    (property "Value" "PWR_FLAG" (at 52.705 85.09 0)
+      (effects (font (size 1.27 1.27)) hide)
+    )
+    (property "Footprint" "" (at 52.705 89.535 0)
+      (effects (font (size 1.27 1.27)) hide)
+    )
+    (property "Datasheet" "~" (at 52.705 89.535 0)
+      (effects (font (size 1.27 1.27)) hide)
+    )
+    (pin "1")
+    (instances
+      (project "100w BLDC Motor Controller Pathfinder"
+        (path "/bd5e620c-77b3-46f1-a718-89cd1182fd75"
           (reference "#FLG02") (unit 1)
+        )
+        (path "/bd5e620c-77b3-46f1-a718-89cd1182fd75/86cdd35b-a858-4f37-a673-ec7a499e55c2"
+          (reference "#FLG05") (unit 1)
         )
       )
@@
         )
       )
+    )
+  )
+  (symbol (lib_id "power:PWR_FLAG") (at 86.36 42.545 0) (unit 1)
+    (in_bom yes) (on_board yes) (dnp no) (fields_autoplaced)
+    (property "Reference" "#FLG02" (at 86.36 40.64 0)
+      (effects (font (size 1.27 1.27)) hide)
+    )
+    (property "Value" "PWR_FLAG" (at 86.36 38.1 0)
+      (effects (font (size 1.27 1.27)) hide)
+    )
+    (property "Footprint" "" (at 86.36 42.545 0)
+      (effects (font (size 1.27 1.27)) hide)
+    )
+    (property "Datasheet" "~" (at 86.36 42.545 0)
+      (effects (font (size 1.27 1.27)) hide)
+    )
+    (pin "1")
+    (instances
+      (project "100w BLDC Motor Controller Pathfinder"
+        (path "/bd5e620c-77b3-46f1-a718-89cd1182fd75"
+          (reference "#FLG02") (unit 1)
+        )
+        (path "/bd5e620c-77b3-46f1-a718-89cd1182fd75/86cdd35b-a858-4f37-a673-ec7a499e55c2"
+          (reference "#FLG04") (unit 1)
+        )
+      )

Commit message: Rev: 0.1
Other:
- note added: "Battery connection"
- company: (none) -> SCS
- title: (none) -> 100w BLDC Motor Controller Pathfinder
- moved on the sheet: C15, C16, C17, C18, C19, C20, C23, D1, D2, J8, L1, R10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

Commit message: .
Parts:
- added D6: LED, LED_SMD:LED_0603_1608Metric, symbol Device:LED
- added R15: 470, symbol Device:R
Connections:
- net +3V3: now also R15.2
- net GND: now also D6.1 (K)
- new net: D6.2 (A), R15.1
Other:
- note added: "3.3v indicator"
- note added: "Voltage Divider"
- note removed: "Voltage Dicider"
- moved on the sheet: R10, R11
